File: eagle/stm32_T12+858D.sch (EAGLE design)
At the start: 79 parts, among them IC1 REG1117, IC2 AD823, IC3 LM328, T1 BTA41 600B, U1 AT24C32A

Commit message: Add files via upload
Parts:
- R24: value 470k -> 100k
- S2: value MODE -> AUTO
Connections:
- removed net N$38: JP2.3, S1.2, U$1.PA8
- net N$36: now also JP2.3, S1.2, U$1.PA8; no longer U$1.PA15
Other:
- moved on the sheet: BZ, R31, R32, S2, VT5

Commit message: Add files via upload
Parts:
- added R39, R40, R41: 100k, rcl:R-EU_0204/5
Connections:
- new net N$64: JP5.4, R40.1, R41.2, TILT.2
- new net N$65: R39.2, U$1.PA8
- net +3V3: now also R40.2
- net N$36: now also R39.1; no longer U$1.PA8
- net N$63: now also R41.1; no longer JP5.4, TILT.2
Other:
- moved on the sheet: R14

Commit message: Add files via upload
Parts:
- IC3: value LM328 -> LM358
Changed lines of the file:
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@@
 <part name="P+4" library="supply1" library_urn="urn:adsk.eagle:library:371" deviceset="+24V" device=""/>
 <part name="R32" library="rcl" library_urn="urn:adsk.eagle:library:334" deviceset="R-EU_" device="0204/5" package3d_urn="urn:adsk.eagle:package:23488/1" value="100"/>
-<part name="IC3" library="linear" library_urn="urn:adsk.eagle:library:262" deviceset="MCP602" device="P" package3d_urn="urn:adsk.eagle:package:16409/2" value="LM328"/>
+<part name="IC3" library="linear" library_urn="urn:adsk.eagle:library:262" deviceset="MCP602" device="P" package3d_urn="urn:adsk.eagle:package:16409/2" value="LM358"/>
 <part name="IC2" library="linear" library_urn="urn:adsk.eagle:library:262" deviceset="MCP602" device="P" package3d_urn="urn:adsk.eagle:package:16409/2" value="AD823"/>
 <part name="GND14" library="supply1" library_urn="urn:adsk.eagle:library:371" deviceset="GND" device=""/>
