File: eagle/stm32_T12+858D_v4.sch (EAGLE design)
At the start: 93 parts, among them IC1 REG1117, IC2 AD823, IC3 LM328, K1 351, T1 BTA41 600B, U1 AT24C32A

Commit message: Add files via upload
Parts:
- JP5: value Amb+tilt -> TILT+AMBIENT; device pinhead:PINHD-1X4 -> pinhead:PINHD-1X2
Connections:
- net N$16 renamed V+
- removed net N$34: JP1.2, R13.2, R9.2
- new net V-: JP1.2, R13.2, R38.1, R9.2, TILT.1
- net GND: no longer JP5.2, JP5.3, R38.1, TILT.1
- net N$29: now also JP5.2; no longer JP5.1
- net N$64: now also JP5.1; no longer JP5.4

Commit message: Add files via upload
Connections:
- removed net N$40: B1.AC2
- net N$73: now also B1.AC2
Changed lines of the file:
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@@
-</segment>
-</net>
-<net name="N$40" class="0">
-<segment>
-<pinref part="B1" gate="1" pin="AC2"/>
-<wire x1="-15.24" y1="-10.16" x2="-17.78" y2="-10.16" width="0.1524" layer="91"/>
 </segment>
 </net>
@@
 <wire x1="-83.82" y1="-27.94" x2="-83.82" y2="-33.02" width="0.1524" layer="91"/>
 <junction x="-83.82" y="-27.94"/>
-</segment>
-</net>
+<pinref part="B1" gate="1" pin="AC2"/>
+<wire x1="-17.78" y1="-10.16" x2="-15.24" y2="-10.16" width="0.1524" layer="91"/>
+<wire x1="-15.24" y1="-10.16" x2="-15.24" y2="2.54" width="0.1524" layer="91"/>
+<wire x1="-15.24" y1="2.54" x2="-83.82" y2="2.54" width="0.1524" layer="91"/>
+<junction x="-83.82" y="2.54"/>
+</segment>
+</net>
